File: hardware/Daughterboard_Channel/ChannelStrip/ChannelStrip.kicad_pcb (KiCad board)
At the start: 2 copper layers, 40 x 100 mm, 9 parts, among them J1 Conn_01x10, SW1 SW_Push, U1 CD74HC4067M

Commit message: sevelaluz
Parts:
- added H1: MountingHole_Pad, MountingHole:MountingHole_2.2mm_M2_Pad_Via, F.Cu at (162.3, 140.9)
- added H2: MountingHole_Pad, MountingHole:MountingHole_2.2mm_M2_Pad_Via, F.Cu at (126.5, 51.0)
- added H3: MountingHole_Pad, MountingHole:MountingHole_2.2mm_M2_Pad_Via, F.Cu at (126.6, 141.0)
- added H4: MountingHole_Pad, MountingHole:MountingHole_2.2mm_M2_Pad_Via, F.Cu at (162.3, 51.0)
- moved J1 22.9 mm to (132.6, 140.4), turned to 180 degrees
- moved R1 8.87 mm to (149.8, 139.4), turned to 180 degrees
- moved FADER1 4.44 mm to (155.6, 129.0)
- moved SW1 2.42 mm to (158.2, 134.4), turned to -90 degrees
Routing:
- net +3V3: track 0.00 -> 113.6 mm
- net /C4: track 0.00 -> 69.5 mm
- net /C3: track 0.00 -> 53.5 mm
- net /C2: track 0.00 -> 38.1 mm
- net /C1: track 0.00 -> 23.3 mm
- net /C0: track 0.00 -> 21.9 mm, vias 0 -> 1
- net /S3: track 0.00 -> 19.6 mm, vias 0 -> 2
- net Net-(U1-I5): track 0.00 -> 18.9 mm, vias 0 -> 2
- net /S2: track 0.00 -> 17.4 mm
- net Net-(R1-Pad1): track 0.00 -> 11.1 mm
- net /S1: track 0.00 -> 7.04 mm
- net /SIG: track 0.00 -> 6.89 mm
- net /S0: track 0.00 -> 6.36 mm, vias 0 -> 2
- net GND: track 0.00 -> 0.30 mm, vias 0 -> 2
- added copper zone on B.Cu, net GND
Other:
- board size 40 x 100 mm -> 45.8 x 100 mm
