File: hardware/Daughterboard_Channel/ChannelStrip/ChannelStrip.kicad_sch (KiCad schematic)
At the start: 9 parts, among them J1 Conn_01x10, SW1 SW_Push, U1 CD74HC4067M

Commit message: sevelaluz
Parts:
- added H1, H2, H3, H4: MountingHole_Pad, MountingHole:MountingHole_2.2mm_M2_Pad_Via, symbol Mechanical:MountingHole_Pad
Changed lines of the file:
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@@
     (effects (font (size 1.27 1.27)) (justify left bottom))
+  )
+  (symbol (lib_id "Mechanical:MountingHole_Pad") (at 54.61 153.67 0) (unit 1)
+    (in_bom yes) (on_board yes) (dnp no) (fields_autoplaced)
+    (property "Reference" "H3" (at 57.15 151.13 0)
+      (effects (font (size 1.27 1.27)) (justify left))
+    )
+    (property "Value" "MountingHole_Pad" (at 57.15 153.67 0)
+      (effects (font (size 1.27 1.27)) (justify left))
+    )
+    (property "Footprint" "MountingHole:MountingHole_2.2mm_M2_Pad_Via" (at 54.61 153.67 0)
+      (effects (font (size 1.27 1.27)) hide)
+    )
+    (property "Datasheet" "~" (at 54.61 153.67 0)
+      (effects (font (size 1.27 1.27)) hide)
+    )
+    (pin "1")
+    (instances
+      (project "ChannelStrip"
+        (path "/1f25699a-42ae-42c6-b63f-3ad17103a86e"
+          (reference "H3") (unit 1)
+        )
+      )
+    )
   )
   (symbol (lib_id "power:GND") (at 104.14 121.92 180) (unit 1)
@@
     )
   )
+  (symbol (lib_id "Mechanical:MountingHole_Pad") (at 54.61 137.16 0) (unit 1)
+    (in_bom yes) (on_board yes) (dnp no) (fields_autoplaced)
+    (property "Reference" "H1" (at 57.15 134.62 0)
+      (effects (font (size 1.27 1.27)) (justify left))
+    )
+    (property "Value" "MountingHole_Pad" (at 57.15 137.16 0)
+      (effects (font (size 1.27 1.27)) (justify left))
+    )
+    (property "Footprint" "MountingHole:MountingHole_2.2mm_M2_Pad_Via" (at 54.61 137.16 0)
+      (effects (font (size 1.27 1.27)) hide)
+    )
+    (property "Datasheet" "~" (at 54.61 137.16 0)
+      (effects (font (size 1.27 1.27)) hide)
+    )
+    (pin "1")
+    (instances
+      (project "ChannelStrip"
+        (path "/1f25699a-42ae-42c6-b63f-3ad17103a86e"
+          (reference "H1") (unit 1)
+        )
+      )
+    )
+  )
   (symbol (lib_id "power:GND") (at 194.31 107.95 0) (unit 1)
     (in_bom yes) (on_board yes) (dnp no)
@@
         (path "/1f25699a-42ae-42c6-b63f-3ad17103a86e"
           (reference "#PWR010") (unit 1)
+        )
+      )
+    )
+  )
+  (symbol (lib_id "Mechanical:MountingHole_Pad") (at 54.61 162.56 0) (unit 1)
+    (in_bom yes) (on_board yes) (dnp no) (fields_autoplaced)
+    (property "Reference" "H4" (at 57.15 160.02 0)
+      (effects (font (size 1.27 1.27)) (justify left))
+    )
+    (property "Value" "MountingHole_Pad" (at 57.15 162.56 0)
+      (effects (font (size 1.27 1.27)) (justify left))
+    )
+    (property "Footprint" "MountingHole:MountingHole_2.2mm_M2_Pad_Via" (at 54.61 162.56 0)
+      (effects (font (size 1.27 1.27)) hide)
+    )
+    (property "Datasheet" "~" (at 54.61 162.56 0)
+      (effects (font (size 1.27 1.27)) hide)
+    )
+    (pin "1")
+    (instances
+      (project "ChannelStrip"
+        (path "/1f25699a-42ae-42c6-b63f-3ad17103a86e"
+          (reference "H4") (unit 1)
         )
       )
@@
         )
       )
+    )
+  )
+  (symbol (lib_id "Mechanical:MountingHole_Pad") (at 54.61 144.78 0) (unit 1)
+    (in_bom yes) (on_board yes) (dnp no) (fields_autoplaced)
+    (property "Reference" "H2" (at 57.15 142.24 0)
+      (effects (font (size 1.27 1.27)) (justify left))
+    )
+    (property "Value" "MountingHole_Pad" (at 57.15 144.78 0)
+      (effects (font (size 1.27 1.27)) (justify left))
+    )
+    (property "Footprint" "MountingHole:MountingHole_2.2mm_M2_Pad_Via" (at 54.61 144.78 0)
+      (effects (font (size 1.27 1.27)) hide)
+    )
+    (property "Datasheet" "~" (at 54.61 144.78 0)
+      (effects (font (size 1.27 1.27)) hide)
+    )
+    (pin "1")
+    (instances
+      (project "ChannelStrip"
+        (path "/1f25699a-42ae-42c6-b63f-3ad17103a86e"
+          (reference "H2") (unit 1)
+        )
+      )

Commit message: poniendorden
Parts:
- H1: value MountingHole_Pad -> MountingHole; symbol Mechanical:MountingHole_Pad -> Mechanical:MountingHole
- H2, H3, H4: symbol Mechanical:MountingHole_Pad -> Mechanical:MountingHole
Other:
- note added: "EXPANSION PORTS"
- note added: "FADERS & POTS"
- note added: "HOLES"
- note added: "MUX"
- note added: "PWR_FLAGS"
- company: (none) -> Ruben Puig Mur
- title: (none) -> RootMixer Module
- moved on the sheet: FADER1, J1, POT1, POT2, POT3, POT4, R1, SW1, U1
