File: hardware/Motherboard/Motherboard/Motherboard.kicad_pcb (KiCad board)
At the start: 2 copper layers, 80 x 50 mm, 21 parts, among them J1 USB_C_Receptacle_USB2.0_16P, J2 Conn_01x04, U1 STM32F411CEUx, U2 AP2112K-3.3, Y1 25MHz

Commit message: letsfirm
Parts:
- moved C7 98.1 mm to (146.1, 93.7)
- moved C8 98.1 mm to (152.6, 105.1)
- moved J_CH1 98.1 mm to (177.1, 115.8)
- moved J_CH2 98.1 mm to (161.1, 115.8)
- moved J_CH4 98.1 mm to (128.1, 115.8)
- moved U1 98.1 mm to (149.6, 99.4)
- moved C1 98.1 mm to (155.2, 100.0)
- moved C2 98.1 mm to (155.2, 101.5)
- moved C3 98.1 mm to (125.0, 84.6)
- moved C4 98.1 mm to (133.7, 87.8)
- moved C5 98.1 mm to (155.2, 98.5)
- moved J2 98.1 mm to (133.1, 105.1)
- moved R2 98.1 mm to (116.9, 86.1)
- moved Y1 98.1 mm to (159.2, 100.7)
- moved C6 98.1 mm to (143.8, 102.2)
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Other:
- board text added: "RootMixer Motherboard v1.0"
- board text added: "niños con los sueños rotos"

Commit message: yoqse2
Parts:
- added H1: MountingHole, MountingHole:MountingHole_2.2mm_M2_Pad_Via, F.Cu at (187.4, 79.7)
- added H2: MountingHole, MountingHole:MountingHole_2.2mm_M2_Pad_Via, F.Cu at (129.0, 79.7)
- added H3: MountingHole, MountingHole:MountingHole_2.2mm_M2_Pad_Via, F.Cu at (117.5, 119.7)
- added H4: MountingHole, MountingHole:MountingHole_2.2mm_M2_Pad_Via, F.Cu at (187.4, 119.7)
- added H5: MountingHole, MountingHole:MountingHole_2.2mm_M2_Pad_Via, F.Cu at (117.5, 93.0)
Routing:
- net GND: vias 22 -> 24

Commit message: poniendorden
Routing:
- net GND: vias 24 -> 22
Changed lines of the file:
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@@
       (drillshape 0)
       (scaleselection 1)
-      (outputdirectory "")
+      (outputdirectory "../Motherboard_Gerber/")
     )
   )
@@
   (via (at 129.396331 85.937161) (size 0.6) (drill 0.3) (layers "F.Cu" "B.Cu") (net 2))
   (via (at 130.55 114.0425) (size 0.6) (drill 0.3) (layers "F.Cu" "B.Cu") (net 2))
-  (via (at 130.989725 78.975714) (size 0.6) (drill 0.3) (layers "F.Cu" "B.Cu") (net 2))
   (via (at 166.11 120.3925) (size 0.6) (drill 0.3) (layers "F.Cu" "B.Cu") (net 2))
   (via (at 180.08 114.0425) (size 0.6) (drill 0.3) (layers "F.Cu" "B.Cu") (net 2))
@@
   (via (at 126.74 115.3125) (size 0.6) (drill 0.3) (layers "F.Cu" "B.Cu") (net 2))
   (via (at 162.3 100.0725) (size 0.6) (drill 0.3) (layers "F.Cu" "B.Cu") (net 2))
-  (via (at 116.411275 94.882433) (size 0.6) (drill 0.3) (layers "F.Cu" "B.Cu") (net 2))
   (via (at 152.14 107.6925) (size 0.6) (drill 0.3) (layers "F.Cu" "B.Cu") (net 2))
   (via (at 116.365 87.3575) (size 0.6) (drill 0.3) (layers "F.Cu" "B.Cu") (net 2))
